Commit message: add RS-Bpearl

File: robosense_description/urdf/HDL-32E.urdf.xacro (robot description, xacro)
@@ -12,7 +12,5 @@
         <mass value="1.0"/>
         <origin xyz="0 0 0.07212"/>
-        <inertia ixx="${(1.0 * (3.0*0.04267*0.04267 + 0.14424*0.14424)) / 12.0}" ixy="0" ixz="0"
-          iyy="${(1.0 * (3.0*0.04267*0.04267 + 0.14424*0.14424)) / 12.0}" iyz="0"
-          izz="${0.5 * 1.0 * (0.04267*0.04267)}"/>
+        <inertia ixx="${(1.0 * (3.0*0.04267*0.04267 + 0.14424*0.14424)) / 12.0}" ixy="0" ixz="0" iyy="${(1.0 * (3.0*0.04267*0.04267 + 0.14424*0.14424)) / 12.0}" iyz="0" izz="${0.5 * 1.0 * (0.04267*0.04267)}"/>
       </inertial>
       <visual>
@@ -28,5 +26,5 @@
       </collision>
     </link>
-    <joint name="${name}_base_scan_joint" type="fixed" >
+    <joint name="${name}_base_scan_joint" type="fixed">
       <origin xyz="0 0 0.09081" rpy="0 0 0" />
       <parent link="${name}_base_link" />
