Commit message: add example(do not work)

File: robosense_description/urdf/RS-Bpearl.urdf.xacro (robot description, xacro)
@@ -63,5 +63,5 @@
                 <resolution>1</resolution>
                 <min_angle> ${0.0*M_PI/180.0}</min_angle>
-                <max_angle> ${81.0*M_PI/180.0}</max_angle>
+                <max_angle> ${82.0*M_PI/180.0}</max_angle>
                 <!-- <min_angle>-${0.0*M_PI/180.0}</min_angle>
                 <max_angle> ${90.0*M_PI/180.0}</max_angle> -->

File: robosense_description/urdf/example.urdf.xacro (robot description, xacro)
@@ -6,10 +6,10 @@
   <link name="base_footprint" />
   <!-- Base Link -->
-  <joint name="footprint" type="fixed" >
-   <parent link="base_footprint" />
+  <joint name="footprint" type="fixed">
+    <parent link="base_footprint" />
     <child link="base_link" />
     <origin xyz="0 0 0.05" rpy="0 0 0" />
   </joint>
-  <link name="base_link" >
+  <link name="base_link">
     <visual>
       <geometry>
@@ -25,16 +25,19 @@
       <origin xyz="0 0 0"/>
       <mass value="10"/>
-      <inertia ixx="3.0" ixy="0.0" ixz="0.0"
-               iyy="3.0" iyz="0.0"
-               izz="3.0" />
+      <inertia ixx="3.0" ixy="0.0" ixz="0.0" iyy="3.0" iyz="0.0" izz="3.0" />
     </inertial>
   </link>
-  <xacro:include filename="$(find velodyne_description)/urdf/VLP-16.urdf.xacro"/>
+  <!-- <xacro:include filename="$(find robosense_description)/urdf/VLP-16.urdf.xacro"/>
   <xacro:VLP-16 parent="base_link" name="velodyne" topic="/velodyne_points" hz="10" samples="440" gpu="${gpu}">
     <origin xyz="0 0 0.4" rpy="0 0 0" />
   </xacro:VLP-16>
-  <xacro:include filename="$(find velodyne_description)/urdf/HDL-32E.urdf.xacro"/>
+  <xacro:include filename="$(find robosense_description)/urdf/HDL-32E.urdf.xacro"/>
   <xacro:HDL-32E parent="base_link" name="velodyne2" topic="/velodyne_points2" hz="10" samples="220" gpu="${gpu}">
     <origin xyz="0 0 0.6" rpy="0 0 0" />
-  </xacro:HDL-32E>
+  </xacro:HDL-32E> -->
+  <!-- RS-Bpearl -->
+  <xacro:include filename="$(find robosense_description)/urdf/RS-Bpearl.urdf.xacro"/>
+  <xacro:RS-Bpearl parent="base_link" name="robosense" topic="/rs_points" hz="20" samples="900" gpu="true">
+    <origin xyz="0 0 0.2" rpy="0 0 0" />
+  </xacro:RS-Bpearl>
 </robot>
